File: PCB Desing/G22V3.brd (EAGLE design)
At the start: 120.3 x 45.7 mm, 20 parts, among them X2 5566-4

Commit message: V4 donete
Parts:
- moved 12V 34.5 mm to (80.0, 14.0)
- moved X2 25.4 mm to (63.5, 10.2)
- moved CANBUS 1.27 mm to (92.5, 34.8)
Routing:
- net VIN: track 111.5 -> 78.8 mm
- net D3: track 72.1 -> 48.5 mm
- net D2: track 74.7 -> 52.1 mm
- net GND: track 266.5 -> 249.5 mm
- net VCC: track 126.1 -> 127.3 mm
- net SCK: track 85.6 -> 86.8 mm
- net MOSI: track 67.8 -> 69.1 mm
- net MISO: track 68.5 -> 69.8 mm
Other:
- board size 120.3 x 45.7 mm -> 96.2 x 45.7 mm
